File: Hardware/Project1/LSM6DS3_Breakout.brd (EAGLE design)
At the start: 25.4 x 25.4 mm, 31 parts

Commit message: ready for proto
Parts:
- added R1, R2: 4.7K, SparkFun-Resistors:0603-RES
- SJ5: value S_MODE -> INT2_JP; device SparkFun-Passives:PAD-JUMPER-3-2OF3_NC_BY_PASTE_YES_SILK_FULL_BOX -> SparkFun-Passives:PAD-JUMPER-2-NC_BY_PASTE_YES_SILK
- SJ6: value INT2_JP -> S_MODE; device SparkFun-Passives:PAD-JUMPER-2-NC_BY_PASTE_YES_SILK -> SparkFun-Passives:PAD-JUMPER-3-2OF3_NC_BY_PASTE_YES_SILK_FULL_BOX
- STANDOFF1, STANDOFF2, STANDOFF3, STANDOFF4: value (none) -> STAND-OFF
- moved SJ5 10.8 mm to (10.8, 7.62), turned to 270 degrees
- moved SJ6 10.8 mm to (14.0, 17.9), turned to 0 degrees
- moved TP2 1.60 mm to (17.1, 12.4)
- moved SJ3 1.59 mm to (19.1, 12.4)
- moved SJ7 1.59 mm to (5.08, 10.6), turned to 270 degrees
- moved LOGO1 1.46 mm to (24.0, 1.91)
- moved LOGO2 1.02 mm to (22.2, 22.4)
- moved L1 0.35 mm to (7.30, 14.0)
- moved U1 0.32 mm to (2.22, 12.7)
- moved SJ2 0.32 mm to (19.1, 14.9)
- moved TP1 0.32 mm to (17.1, 14.9)
- turned STANDOFF1 to 0 degrees
- turned STANDOFF2 to 0 degrees
- turned STANDOFF3 to 0 degrees
- turned STANDOFF4 to 0 degrees
- renumbered U$1 to U2, U$2 to STANDOFF4, U$3 to STANDOFF2, U$4 to STANDOFF3, U$5 to STANDOFF1
Connections:
- net 3.3V: now also R1.2, R2.2, SJ6.3; no longer SJ5.3
- net CS: now also SJ6.2; no longer SJ5.2
- net GND: now also SJ6.1; no longer SJ5.1
- net INT2: now also SJ5.1; no longer SJ6.1
- net N$3: now also SJ5.2; no longer SJ6.2
- net SCL: now also R1.1
- net SDA: now also R2.1
Routing:
- net GND: track 10.3 -> 9.07 mm, vias 16 -> 18
- net SDO/SA0: track 16.9 -> 15.9 mm
- net 3.3V: track 48.0 -> 47.2 mm
- net N$5: track 22.1 -> 22.8 mm
- net SDX: track 5.46 -> 4.80 mm
Other:
- board text added: "VIN(4-12V)"
- board text removed: "VIN+"
