File: Hardware/Project1/LSM6DS3_Breakout.sch (EAGLE design)
At the start: 27 parts

Commit message: ready for proto
Parts:
- added R1, R2: 4.7K, SparkFun-Resistors:4.7KOHM-1/10W-1%(0603)
- added STANDOFF1, STANDOFF2, STANDOFF3, STANDOFF4: STAND-OFF, SparkFun-Electromechanical:STAND-OFF
- SJ5: value S_MODE -> INT2_JP; device SparkFun-Passives:JUMPER-PAD-3-2OF3_NC_BY_PASTE -> SparkFun-Passives:JUMPER-PAD-2-NC_BY_PASTE
- SJ6: value INT2_JP -> S_MODE; device SparkFun-Passives:JUMPER-PAD-2-NC_BY_PASTE -> SparkFun-Passives:JUMPER-PAD-3-2OF3_NC_BY_PASTE
- renumbered U$1 to U2
Connections:
- net 3.3V: now also R1.2, R2.2, SJ6.3; no longer SJ5.3
- net CS: now also SJ6.2; no longer SJ5.2
- net GND: now also SJ6.1; no longer SJ5.1
- net INT2: now also SJ5.1; no longer SJ6.1
- net N$3: now also SJ5.2; no longer SJ6.2
- net SCL: now also R1.1
- net SDA: now also R2.1
Other:
- note added: "Power supply options 1. Supply 1.8 to 3.3V for power and IO 2. Supply through the regulator for 3.3V operation"
- note added: "Solder jumper selections SJ1 selects LSB of I2C SJ2 allows disconnect of SCX for I2C master or aux SPI SJ3 allows disconnect of SDX for I2C master of aux SPI SJ4 and SJ5 allow disconnect of INT pins for alternate header usage SJ6 selects I2C or SPI mode"
- note removed: "Supply 1.8 to 3.3V for power and IO, OR supply through the regulator for 3.3V operation"
- moved on the sheet: JP1, SJ4
