File: Hardware/LSM6DS3_Breakout.brd (EAGLE design)
At the start: 30.5 x 25.4 mm, 29 parts, among them U2 LSM6DS3DOT_INDICATION

Commit message: v03 commit
Parts:
- removed JP10: INT1, SparkFun-Connectors:1X01
- removed JP4: GP1, SparkFun-Connectors:1X01
- removed JP5: GP2, SparkFun-Connectors:1X01
- removed JP6: OCS, SparkFun-Connectors:1X01
- removed JP7: INT2, SparkFun-Connectors:1X01
- removed JP8: SDx, SparkFun-Connectors:1X01
- removed JP9: SCx, SparkFun-Connectors:1X01
- removed SJ6: S_MODE, SparkFun-Passives:PAD-JUMPER-3-2OF3_NC_BY_PASTE_YES_SILK_FULL_BOX
- added JP11: GND, SparkFun-Connectors:1X01
- added JP2: 3.3V, SparkFun-Connectors:1X01
- added SJ3, SJ4: JUMPER-PAD-2-NC_BY_TRACE, SparkFun-Passives:PAD-JUMPER-2-NC_BY_TRACE_YES_SILK
- JP3: value SDO -> IO; device SparkFun-Connectors:1X01 -> SparkFun-Connectors:1X05
- LOGO1: value SFE_LOGO_NAME_FLAME.1_INCH -> SFE_LOGO_FLAME.2_INCH; device SparkFun-Aesthetics:SFE_LOGO_NAME_FLAME_.1 -> SparkFun-Aesthetics:SFE_LOGO_FLAME_.2
- LOGO3: value SFE_LOGO_FLAME.6_INCH -> SFE_LOGO_NAME_FLAME.1_INCH; device SparkFun-Aesthetics:SFE_LOGO_FLAME_.6 -> SparkFun-Aesthetics:SFE_LOGO_NAME_FLAME_.1
- R3: value 4.7K -> 10K
- SJ1: value I2C ADDR LSB -> (none)
- SJ2: device SparkFun-Passives:PAD-JUMPER-3-NC_BY_PASTE_YES_SILK_FULL_BOX -> SparkFun-Passives:PAD-JUMPER-3-3OF3_NC_BY_TRACE_YES_SILK_FULL_BOX
- U2: value LSM6DS3DOT_INDICATION -> LSM6DS3
- moved LOGO2 32.3 mm to (2.54, 2.06), turned to 0 degrees
- moved JP3 15.5 mm to (6.35, 21.6)
- moved LOGO1 14.4 mm to (17.2, 17.1), turned to 0 degrees
- moved R3 10.4 mm to (15.2, 15.2), turned to 180 degrees
- moved JP1 10.2 mm to (19.1, 1.27), turned to 180 degrees
- moved LOGO3 9.88 mm to (19.3, 8.81), turned to 0 degrees
- moved FID2 6.84 mm to (21.6, 2.54)
- moved R2 6.32 mm to (7.62, 7.46)
- moved FRAME1 5.68 mm to (-19.1, -29.2)
- moved SJ1 4.71 mm to (17.6, 11.4), turned to 90 degrees
- moved STANDOFF1 4.58 mm to (2.54, 16.5)
- moved STANDOFF3 4.58 mm to (20.3, 16.5)
- moved U2 4.02 mm to (11.4, 11.4)
- moved C4 3.86 mm to (11.4, 15.2)
- moved L1 3.86 mm to (7.62, 15.2), turned to 180 degrees
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Connections:
- net N$1 renamed VDD
- removed net N$2: JP6.1, U2.10
- removed net N$3: JP1.5, JP4.1
- removed net N$4: JP1.6, JP5.1
- removed net N$7: R3.1, SJ6.3
- new net OCS: JP3.3, U2.10
- net 3.3V: now also JP1.5, JP2.1; no longer JP1.3
- net CS: now also JP1.1, R3.1; no longer SJ6.2
- net GND: now also JP1.6, JP11.1, SJ3.1, SJ4.1; no longer JP1.4, SJ6.1
- net INT1: now also JP3.2; no longer JP10.1
- net INT2: now also JP3.1; no longer JP7.1
- net SCL: now also JP1.3; no longer JP1.1
- net SCX: now also JP3.4, SJ4.2; no longer JP9.1
- net SDA: now also JP1.4; no longer JP1.2
- net SDO/SA0: now also JP1.2; no longer JP3.1
- net SDX: now also JP3.5, SJ3.2; no longer JP8.1
Routing:
- net N$2: track 20.7 -> 0.00 mm, vias 1 -> 0
- net GND: track 3.81 -> 24.3 mm
- net CS: track 11.4 -> 31.4 mm
- net OCS: track 0.00 -> 18.6 mm, vias 0 -> 2
- net 3.3V: track 62.8 -> 48.7 mm
- net SDA: track 23.6 -> 13.4 mm
- net SCL: track 22.0 -> 13.6 mm
- net N$5: track 2.38 -> 8.73 mm, vias 0 -> 1
- net N$3: track 5.08 -> 0.00 mm
- net N$4: track 5.08 -> 0.00 mm
- net N$6: track 2.38 -> 5.72 mm, vias 0 -> 1
- net INT2: track 17.3 -> 14.5 mm, vias 1 -> 2
- net INT1: track 14.7 -> 12.0 mm, vias 0 -> 2
- net SCX: track 14.3 -> 11.8 mm, vias 0 -> 1
- net VDD: track 3.91 -> 6.11 mm
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Other:
- board size 30.5 x 25.4 mm -> 22.9 x 22.9 mm
- board text added: "CS"
- board text added: "LSM6DS3"
- board text added: "OPEN FOR SPI"
- board text added: "PU EN"
- board text added: "SDA/SDI"
- board text added: "SDO/SA0"
- board text added: "v03"
- board text removed: "GP1"
- board text removed: "GP2"
- board text removed: "I2C"
- board text removed: "LSM6DS3 Breakout Board"
- board text removed: "PULLUP"
- board text removed: "SDO"
- board text removed: "SERIAL"
- board text removed: "SPI"
- board text removed: "v02"
