File: Hardware/LSM6DS3_Breakout.sch (EAGLE design)
At the start: 25 parts, among them U2 LSM6DS3

Commit message: Fixed silk for redboards
Parts:
- FRAME1: VERSION v03 -> v10
- JP1: device SparkFun-Connectors:M06SILK_FEMALE_PTH -> SparkFun-Connectors:M06NO_SILK_YES_STOP
- JP11, JP2: device SparkFun-Connectors:M01PTH -> SparkFun-Connectors:M01PTH_NO_SILK_YES_STOP
Changed lines of the file:
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@@
 <part name="FRAME1" library="SparkFun-Aesthetics" deviceset="FRAME-LETTER" device="">
 <attribute name="DESIGNER" value="Marshall Taylor"/>
-<attribute name="VERSION" value="v03"/>
+<attribute name="VERSION" value="v10"/>
 </part>
 <part name="U2" library="LSM6DS3" deviceset="LSM6DS3" device="DOT_INDICATION" value="LSM6DS3"/>
@@
 <part name="R3" library="SparkFun-Resistors" deviceset="10KOHM-1/10W-1%(0603)" device="0603" value="10K"/>
 <part name="SJ2" library="SparkFun-Passives" deviceset="JUMPER-PAD-3-NC_BY_TRACE" device="" value="S_MODE"/>
-<part name="JP1" library="SparkFun-Connectors" deviceset="M06" device="SILK_FEMALE_PTH" value="IO"/>
+<part name="JP1" library="SparkFun-Connectors" deviceset="M06" device="NO_SILK_YES_STOP" value="IO"/>
 <part name="GND1" library="SparkFun-Aesthetics" deviceset="GND" device=""/>
 <part name="GND2" library="SparkFun-Aesthetics" deviceset="GND" device=""/>
 <part name="SJ3" library="SparkFun-Passives" deviceset="JUMPER-PAD-2-NC_BY_TRACE" device=""/>
 <part name="SJ4" library="SparkFun-Passives" deviceset="JUMPER-PAD-2-NC_BY_TRACE" device=""/>
-<part name="JP2" library="SparkFun-Connectors" deviceset="M01" device="PTH" value="3.3V"/>
-<part name="JP11" library="SparkFun-Connectors" deviceset="M01" device="PTH" value="GND"/>
+<part name="JP2" library="SparkFun-Connectors" deviceset="M01" device="PTH_NO_SILK_YES_STOP" value="3.3V"/>
+<part name="JP11" library="SparkFun-Connectors" deviceset="M01" device="PTH_NO_SILK_YES_STOP" value="GND"/>
 <part name="LOGO3" library="SparkFun-Aesthetics" deviceset="SFE_LOGO_NAME_FLAME" device=".1_INCH" value="SFE_LOGO_NAME_FLAME.1_INCH"/>
 <part name="JP3" library="SparkFun-Connectors" deviceset="M05" device="PTH" value="IO"/>
@@
 <segment>
 <pinref part="U2" gate="G$1" pin="CS"/>
-<label x="120.142" y="112.014" size="1.27" layer="95" font="vector" ratio="15"/>
+<label x="120.142" y="112.014" size="1.27" layer="95" font="vector"/>
 <wire x1="106.68" y1="111.76" x2="124.46" y2="111.76" width="0.1524" layer="91"/>
 <wire x1="124.46" y1="111.76" x2="124.46" y2="116.84" width="0.1524" layer="91"/>
